File: pcb/smol-slime-xiao.kicad_pcb (KiCad board)
At the start: 4 copper layers, 20 x 23.5 mm, 15 parts, among them J1 Battery_Terminal, J2 Charger_Connecter, J3 Conn_01x01, J4 Conn_01x01, SW1 Power_Switch, U1 ICM-45686, U3 1532H, U4 XIAO-nRF52840-SMD

Commit message: Fix DRC errors
Parts:
- U3: footprint Crystal:Crystal_SMD_3225-4Pin_3.2x2.5mm -> Generic:Crystal_SMD_3225-4Pin_3.2x2.5mm_Silkscreenfix
Routing:
- net Net-(J1-Pin_2): vias 1 -> 0
Changed lines of the file:
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@@
 		)
 		(fp_line
-			(start -3.1 7.4)
-			(end 5.2 7.4)
+			(start -1.4 7.4)
+			(end 3.4 7.4)
 			(stroke
 				(width 0.12)
@@
 		(embedded_fonts no)
 	)
-	(footprint "Crystal:Crystal_SMD_3225-4Pin_3.2x2.5mm"
+	(footprint "Generic:Crystal_SMD_3225-4Pin_3.2x2.5mm_Silkscreenfix"
 		(layer "F.Cu")
 		(at 153.75 94.75 180)
@@
 		(fp_line
 			(start -2.06 1.71)
-			(end 2.06 1.71)
+			(end 1.2 1.71)
 			(stroke
 				(width 0.12)
@@
 		)
 		(fp_line
-			(start -2.06 -1.71)
+			(start -2.06 -0.9)
 			(end -2.06 1.71)
 			(stroke
@@
 		)
 		(property "Value" "ICM-45686"
-			(at 0 -5.25 0)
+			(at 10.5 -3 0)
 			(layer "F.Fab")
 			(effects
@@
 	)
 	(segment
-		(start 149.25 91.5)
-		(end 150.5 92.75)
+		(start 150.5 92.75)
+		(end 150.5 97.5)
 		(width 0.3)
 		(layer "F.Cu")
@@
 	)
 	(segment
-		(start 150.5 92.75)
-		(end 150.5 97.5)
+		(start 149.25 91.5)
+		(end 150.5 92.75)
 		(width 0.3)
 		(layer "F.Cu")
 		(net 27)
 	)
-	(via
-		(at 152.05 99.05)
-		(size 0.5)
-		(drill 0.3)
-		(layers "F.Cu" "B.Cu")
-		(net 27)
-	)
