File: pcb/smol-slime-xiao.kicad_sch (KiCad schematic)
At the start: 15 parts, among them J1 Battery_Terminal, J2 Charger_Connecter, J3 Conn_01x01, J4 Conn_01x01, SW1 Power_Switch, U1 ICM-45686, U3 1532H, U4 XIAO-nRF52840-SMD

Commit message: Consolidate custom KiCad libraries into a single project library
The pcb libs folder had grown into one folder per part, each needing its
own sym-lib-table and fp-lib-table entry. The tables had drifted out of
sync with it: fp-lib-table carried a dead ICM_45686 entry pointing at a
path that never existed, and the SSSS811101 switch symbol was never
registered at all. The vendor downloads also left behind duplicate STEP
files, superseded v5-format footprints, and how-to-import cruft.

All custom symbols now live in libs/smol-biscuits.kicad_sym and all
custom footprints in libs/smol-biscuits.pretty, with STEP models shared
in libs/3dmodels. The two older-format symbols (ICM-45686, SSSS811101)
were converted to the current format during the merge. Schematic and
board references were rewritten to the new smol-biscuits nickname, and
embedded 3D model paths updated to the new locations. Vendor license
files are kept at the libs root. This gives rev 2 one obvious place to
import new parts into.
Parts:
- J1: footprint Generic:JST_PH2_SMT -> smol-biscuits:JST_PH2_SMT
- J2: footprint Generic:PinPads_1x03_P2.54mm -> smol-biscuits:PinPads_1x03_P2.54mm
- J3, J4: footprint Generic:Heat_Pad_1.0x1.0mm -> smol-biscuits:Heat_Pad_1.0x1.0mm
- SW1: footprint SW_SSSS811101:SW_SSSS811101 -> smol-biscuits:SW_SSSS811101
- U1: footprint ICM-45686:IC_ICM-45686 -> smol-biscuits:IC_ICM-45686; symbol ICM-45686:ICM-45686 -> smol-biscuits:ICM-45686
- U2: footprint QMC6309:QMC6309 -> smol-biscuits:QMC6309; symbol QMC6309:QMC6309 -> smol-biscuits:QMC6309
- U3: footprint Generic:Crystal_SMD_3225-4Pin_3.2x2.5mm_Silkscreenfix -> smol-biscuits:Crystal_SMD_3225-4Pin_3.2x2.5mm_Silkscreenfix; symbol 1532H4:1532H4 -> smol-biscuits:1532H4
Changed lines of the file:
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@@
 	)
 	(symbol
-		(lib_id "ICM-45686:ICM-45686")
+		(lib_id "smol-biscuits:ICM-45686")
 		(at 80.01 78.74 0)
 		(unit 1)
@@
 			)
 		)
-		(property "Footprint" "ICM-45686:IC_ICM-45686"
+		(property "Footprint" "smol-biscuits:IC_ICM-45686"
 			(at 80.01 78.74 0)
 			(effects
@@
 			)
 		)
-		(property "Footprint" "Generic:JST_PH2_SMT"
+		(property "Footprint" "smol-biscuits:JST_PH2_SMT"
 			(at 217.17 82.55 0)
 			(effects
@@
 			)
 		)
-		(property "Footprint" "Generic:Heat_Pad_1.0x1.0mm"
+		(property "Footprint" "smol-biscuits:Heat_Pad_1.0x1.0mm"
 			(at 217.17 74.93 0)
 			(effects
@@
 			)
 		)
-		(property "Footprint" "Generic:Heat_Pad_1.0x1.0mm"
+		(property "Footprint" "smol-biscuits:Heat_Pad_1.0x1.0mm"
 			(at 217.17 97.79 0)
 			(effects
@@
 			)
 		)
-		(property "Footprint" "Generic:PinPads_1x03_P2.54mm"
+		(property "Footprint" "smol-biscuits:PinPads_1x03_P2.54mm"
 			(at 217.17 105.41 0)
 			(effects
@@
 	)
 	(symbol
-		(lib_id "QMC6309:QMC6309")
+		(lib_id "smol-biscuits:QMC6309")
 		(at 172.72 130.81 0)
 		(unit 1)
@@
 			)
 		)
-		(property "Footprint" "QMC6309:QMC6309"
+		(property "Footprint" "smol-biscuits:QMC6309"
 			(at 172.72 130.81 0)
 			(effects
@@
 	)
 	(symbol
-		(lib_id "1532H4:1532H4")
+		(lib_id "smol-biscuits:1532H4")
 		(at 161.29 52.07 0)
 		(unit 1)
@@
 			)
 		)
-		(property "Footprint" "Generic:Crystal_SMD_3225-4Pin_3.2x2.5mm_Silkscreenfix"
+		(property "Footprint" "smol-biscuits:Crystal_SMD_3225-4Pin_3.2x2.5mm_Silkscreenfix"
 			(at 161.29 52.07 0)
 			(effects
@@
 			)
 		)
-		(property "Footprint" "SW_SSSS811101:SW_SSSS811101"
+		(property "Footprint" "smol-biscuits:SW_SSSS811101"
 			(at 253.238 95.25 90)
 			(effects
