File: pcb/smol-slime-rev2.kicad_sch (KiCad schematic)
At the start: 48 parts, among them J1 BATTERY, J2 SWD, J3 VTREF_RST, J4 TYPE-C-31-M-17, SW1 TS-1088-AR02016, U1 nPM1300, U2 LSM6DSV16X, U3 QMC6309, U4 nRF52840-QIAA, X1 32MHz CL=8pF

Commit message: Fix C11 value
Parts:
- C11: value 100nF -> 2.2nF
Changed lines of the file:
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@@
 			)
 		)
-		(property "Value" "100nF"
+		(property "Value" "2.2nF"
 			(at 261.62 99.06 0)
 			(show_name no)

Commit message: Fix magnetometer decoupling cap C11 to 2.2 uF
C11 on the QMC6309 VDD was sitting at 2.2 nF in the schematic, a micro
for nano slip that made it a thousand times too small. The QMC6309
datasheet (section 4.3.3 and figure 6) calls for a 2.2 uF low ESR
reservoir capacitor on VDD, sized to supply the set and reset pulses the
sensor fires on every measurement. Changed the value to 2.2 uF and moved
the part to 0603 so it matches the other bulk caps and gets the low ESR
the datasheet asks for.

The support-part map and the shopping list had recorded C11 as 100 nF,
which never matched the schematic, so the cap counts are corrected too:
100 nF is seven parts, 2.2 uF is now two.
Parts:
- C11: value 2.2nF -> 2.2uF; footprint Capacitor_SMD:C_0402_1005Metric -> Capacitor_SMD:C_0603_1608Metric
Changed lines of the file:
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@@
 			)
 		)
-		(property "Value" "2.2nF"
+		(property "Value" "2.2uF"
 			(at 261.62 99.06 0)
 			(show_name no)
@@
 			)
 		)
-		(property "Footprint" "Capacitor_SMD:C_0402_1005Metric"
+		(property "Footprint" "Capacitor_SMD:C_0603_1608Metric"
 			(at 259.08 93.98 0)
 			(hide yes)
